File: boiling_control_system_kicad/arduino_connections.sch (KiCad schematic (older format))
At the start: 26 parts, among them J1 Screw_Terminal_01x02, J2 Screw_Terminal_01x02, K1 SSR-40 DA, SW1 SW_Reed, SW2 SW_Reed, U1 sw_btn, U2 sw_btn, U4 sw_btn, U7 DS18B20

Commit message: fix: kicad project, +archieved
Parts:
- PWR3: symbol test_project-rescue:COMMON_-power_GOST -> arduino_connections-rescue:COMMON_-power_GOST-test_project-rescue
- U1, U2, U4: symbol test_project-rescue:sw_btn-test_project-cache -> arduino_connections-rescue:sw_btn-test_project-cache-test_project-rescue
Changed lines of the file:
@@
 $EndComp
 $Comp
-L test_project-rescue:COMMON_-power_GOST PWR3
+L arduino_connections-rescue:COMMON_-power_GOST-test_project-rescue PWR3
 U 1 1 603BF4BC
 P 3590 2505
@@
 $EndComp
 $Comp
-L test_project-rescue:+12V #PWR01
+L arduino_connections-rescue:+12V-test_project-rescue #PWR01
 U 1 1 604E5161
 P 2800 1385
@@
 $EndComp
 $Comp
-L test_project-rescue:sw_btn-test_project-cache U4
+L arduino_connections-rescue:sw_btn-test_project-cache-test_project-rescue U4
 U 1 1 60588C51
 P 3290 3180
@@
 $EndComp
 $Comp
-L test_project-rescue:sw_btn-test_project-cache U2
+L arduino_connections-rescue:sw_btn-test_project-cache-test_project-rescue U2
 U 1 1 60586A8E
 P 3290 2980
@@
 $EndComp
 $Comp
-L test_project-rescue:sw_btn-test_project-cache U1
+L arduino_connections-rescue:sw_btn-test_project-cache-test_project-rescue U1
 U 1 1 6057E898
 P 3290 2780
@@
 $EndComp
 $Comp
-L test_project-rescue:+12V #PWR02
+L arduino_connections-rescue:+12V-test_project-rescue #PWR02
 U 1 1 604EA431
 P 4365 1380

Commit message: fix: circuit
Connections:
- net labels added: Btn_Cancel_D10, Btn_Down_D9, Btn_Up_D8, Higher_D5, Lower_D4
- net labels removed: D4, D5
- wire segments 71 -> 72
Other:
- moved on the sheet: K1, R1, R2, R3, R4
